Commit message: called method to handle ros service data before rest, to ensure it being called. Modified robot urdf to set correct orientation

File: demconRobot.xacro (robot description, xacro)
@@ -27,4 +27,5 @@
 		<parent link="base_footprint" />
 		<child link="base_link" />
+		<origin rpy="0 0 ${-0.5*M_PI}"/>
 	</joint>
 	<link name="wheelFrontLeft">

Commit message: changed to new filter/fuser,, modified some settings and started on new UI

File: demconRobot.xacro (robot description, xacro)
@@ -23,4 +23,9 @@
 			</material>
 		</visual>
+		<collision>
+			<geometry>
+				<cylinder length="0.2" radius="0.4" />
+			</geometry>
+		</collision>
 	</link>
 	<joint name="base_footprint_joint" type="fixed">
@@ -78,4 +83,14 @@
 		</visual>
 	</link>
+	<link name="base_imu">
+		<visual>
+			<geometry>
+				<box size="0.001 0.001 0.001" />
+			</geometry>
+			<material name="white">
+				<color rgba="1 1 1 1"/>
+			</material>
+		</visual>
+	</link>
 	<joint name="base_to_front_left_wheel" type="fixed">
 		<parent link="base_link"/>
@@ -103,3 +118,8 @@
 		<origin xyz="0 0.18 0" rpy="0 0 ${-0.5*M_PI}"/>
 	</joint>
+	<joint name="base_to_imu" type="fixed">
+		<parent link="base_link"/>
+		<child link="base_imu"/>
+		<origin xyz="0 0 0.001" rpy="0 0 0"/>
+	</joint>
 </robot>
